File: hardware/board/ecoport-bridge-v1/ecoport-bridge-v1.kicad_sch (KiCad schematic)
At the start: 61 parts, among them J1 420B2V12FL0, J2 Conn_01x02, J3 SM04B-SRSS-TB, J4 USB4085-GF-A, J5 Conn_01x02, J6 Connector Wire, J7 B3B-PH-K-S, SW1 RESET, SW2 BOOT, U1 IRM-05-5, U2 TLV75733PDBVR, U3 SP3485EET, U4 USBLC6-2SC6, U5 SN74LV1T34DCKR, U6 ESP32-C6-WROOM-1-N8, U7 USBLC6-2SC6

Commit message: Initial board design  DRC all passes
Parts:
- J3: footprint Snapeda:CONN4_BM04B-SRSS_JST -> Custom:CONN4_BM04B-SRSS_JST
Changed lines of the file:
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@@
 			)
 		)
-		(property "Footprint" "Snapeda:CONN4_BM04B-SRSS_JST"
+		(property "Footprint" "Custom:CONN4_BM04B-SRSS_JST"
 			(at 41.9101 158.75 90)
 			(hide yes)

Commit message: Added fuse
Parts:
- added F1: SF-2410SP050W-2, Samacsys:FUSC6125X236N, symbol Samacsys:SF-2410SP050W-2
Connections:
- net AC_L2: now also F1.1; no longer U1.1 (AC/N)
- new net AC_L2_F: F1.2, U1.1 (AC/N)
Changed lines of the file:
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@@
 	(wire
 		(pts
-			(xy 54.61 53.34) (xy 54.61 69.85)
+			(xy 54.61 53.34) (xy 54.61 71.12)
 		)
 		(stroke
@@
 	(wire
 		(pts
+			(xy 90.17 63.5) (xy 104.14 63.5)
+		)
+		(stroke
+			(width 0)
+			(type default)
+		)
+	)
+	(wire
+		(pts
 			(xy 284.48 180.34) (xy 289.56 180.34)
 		)
@@
 	(wire
 		(pts
-			(xy 57.15 63.5) (xy 104.14 63.5)
+			(xy 57.15 69.85) (xy 67.31 69.85)
 		)
 		(stroke
@@
 	(wire
 		(pts
-			(xy 57.15 58.42) (xy 57.15 63.5)
+			(xy 57.15 58.42) (xy 57.15 69.85)
 		)
 		(stroke
@@
 	(wire
 		(pts
+			(xy 85.09 69.85) (xy 90.17 69.85)
+		)
+		(stroke
+			(width 0)
+			(type default)
+		)
+	)
+	(wire
+		(pts
 			(xy 180.34 58.42) (xy 180.34 60.96)
 		)
@@
 	(wire
 		(pts
+			(xy 90.17 69.85) (xy 90.17 63.5)
+		)
+		(stroke
+			(width 0)
+			(type default)
+		)
+	)
+	(wire
+		(pts
 			(xy 67.31 154.94) (xy 72.39 154.94)
 		)
@@
 		)
 	)
-	(label "AC_L2"
+	(label "AC_L2_F"
 		(at 95.25 63.5 0)
 		(fields_autoplaced yes)
@@
 		)
 	)
+	(label "AC_L2"
+		(at 59.69 69.85 0)
+		(fields_autoplaced yes)
+		(effects
+			(font
+				(size 1.27 1.27)
+			)
+			(justify left bottom)
+		)
+		(property "Netclass" "Mains"
+			(at 59.69 71.12 0)
+			(show_name no)
+			(do_not_autoplace no)
+			(effects
+				(font
+					(size 1.27 1.27)
+					(italic yes)
+				)
+				(justify left)
+			)
+		)
+	)
 	(label "SDA"
 		(at 106.68 152.4 0)
@@
 	)
 	(symbol
+		(lib_id "Samacsys:SF-2410SP050W-2")
+		(at 67.31 69.85 0)
+		(unit 1)
+		(body_style 1)
+		(exclude_from_sim no)
+		(in_bom yes)
+		(on_board yes)
+		(in_pos_files yes)
+		(dnp no)
+		(fields_autoplaced yes)
+		(property "Reference" "F1"
+			(at 76.2 63.5 0)
+			(show_name no)
+			(do_not_autoplace no)
+			(effects
+				(font
+					(size 1.27 1.27)
+				)
+			)
+		)
+		(property "Value" "SF-2410SP050W-2"
+			(at 76.2 66.04 0)
+			(show_name no)
+			(do_not_autoplace no)
+			(effects
+				(font
+					(size 1.27 1.27)
+				)
+			)
+		)
+		(property "Footprint" "Samacsys:FUSC6125X236N"
+			(at 76.2 43.18 0)
+			(hide yes)
+			(show_name no)
+			(do_not_autoplace no)
+			(effects
+				(font
+					(size 1.27 1.27)
+				)
+			)
+		)
+		(property "Datasheet" "https://www.bourns.com/docs/Product-Datasheets/SF-2410SPxxxW.pdf"
+			(at 76.2 45.72 0)
+			(hide yes)
+			(show_name no)
+			(do_not_autoplace no)
+			(effects
+				(font
+					(size 1.27 1.27)
+				)
+			)
+		)
+		(property "Description" "Surface Mount Fuses 0.5A Time Lag 2410 SinglFuse"
+			(at 76.2 48.26 0)
+			(hide yes)
+			(show_name no)
+			(do_not_autoplace no)
+			(effects
+				(font
+					(size 1.27 1.27)
+				)
+			)
+		)
+		(property "Height" "2.36"
+			(at 76.2 50.8 0)
+			(hide yes)
+			(show_name no)
+			(do_not_autoplace no)
+			(effects
+				(font
+					(size 1.27 1.27)
+				)
+			)
+		)
+		(property "Manufacturer_Name" "Bourns"
+			(at 76.2 53.34 0)
+			(hide yes)
+			(show_name no)
+			(do_not_autoplace no)
+			(effects
+				(font
+					(size 1.27 1.27)
+				)
+			)
+		)
+		(property "Manufacturer_Part_Number" "SF-2410SP050W-2"
+			(at 76.2 55.88 0)
+			(hide yes)
+			(show_name no)
+			(do_not_autoplace no)
+			(effects
+				(font
+					(size 1.27 1.27)
+				)
+			)
+		)
+		(property "Mouser Part Number" "652-SF-2410SP050W-2"
+			(at 76.2 58.42 0)
+			(hide yes)
+			(show_name no)
+			(do_not_autoplace no)
+			(effects
+				(font
+					(size 1.27 1.27)
+				)
+			)
+		)
+		(property "Mouser Price/Stock" "https://www.mouser.co.uk/ProductDetail/Bourns/SF-2410SP050W-2?qs=55YtniHzbhAbLtmcAyIlLQ%3D%3D"
+			(at 76.2 60.96 0)
+			(hide yes)
+			(show_name no)
+			(do_not_autoplace no)
+			(effects
+				(font
+					(size 1.27 1.27)
+				)
+			)
+		)
+		(property "Arrow Part Number" "SF-2410SP050W-2"
+			(at 76.2 63.5 0)
+			(hide yes)
+			(show_name no)
+			(do_not_autoplace no)
+			(effects
+				(font
+					(size 1.27 1.27)
+				)
+			)
+		)
+		(property "Arrow Price/Stock" "https://www.arrow.com/en/products/sf-2410sp050w-2/bourns?region=nac"
+			(at 76.2 66.04 0)
+			(hide yes)
+			(show_name no)
+			(do_not_autoplace no)
+			(effects
+				(font
+					(size 1.27 1.27)
+				)
+			)
+		)
+		(pin "1"
+		)
+		(pin "2"
+		)
+		(instances
+			(project "ecoport-bridge-v1"
+				(path "/2df6f809-6dc3-4e88-ae5c-1829baf48336"
+					(reference "F1")
+					(unit 1)
+				)
+			)
+		)
+	)
+	(symbol
 		(lib_name "TestPoint_1")
 		(lib_id "Connector:TestPoint")
@@
 	(symbol
 		(lib_id "power:Earth")
-		(at 54.61 69.85 0)
+		(at 54.61 71.12 0)
 		(unit 1)
 		(body_style 1)
@@
 		(fields_autoplaced yes)
 		(property "Reference" "#PWR03"
-			(at 54.61 76.2 0)
+			(at 54.61 77.47 0)
 			(hide yes)
 			(show_name no)
@@
 		)
 		(property "Value" "Earth"
-			(at 54.61 74.93 0)
+			(at 54.61 76.2 0)
 			(show_name no)
 			(do_not_autoplace no)
@@
 		)
 		(property "Footprint" ""
-			(at 54.61 69.85 0)
+			(at 54.61 71.12 0)
 			(hide yes)
 			(show_name no)
@@
 		)
 		(property "Datasheet" ""
-			(at 54.61 69.85 0)
+			(at 54.61 71.12 0)
 			(hide yes)
 			(show_name no)
@@
 		)
 		(property "Description" "Power symbol creates a global label with name \"Earth\""
-			(at 54.61 69.85 0)
+			(at 54.61 71.12 0)
 			(hide yes)
 			(show_name no)

Commit message: added usb power and reorganized assets
Parts:
- added C16: 1µF, Capacitor_SMD:C_0603_1608Metric, symbol Device:C
- added U8: LM66100DCKR, Package_TO_SOT_SMD:SOT-363_SC-70-6, symbol Power_Management:LM66100DCK
- F1: footprint Samacsys:FUSC6125X236N -> Custom:FUSC6125X236N; symbol Samacsys:SF-2410SP050W-2 -> Custom:SF-2410SP050W-2
- J4: symbol EasyEDA:USB4085-GF-A -> Custom:USB4085-GF-A
- J7: footprint Snapeda:JST_B3B-PH-K-S -> Custom:JST_B3B-PH-K-S; symbol SnapEDA:B3B-PH-K-S -> Custom:B3B-PH-K-S
- SW1, SW2: footprint Snapeda:SW_TS04-66-50-BK-260-SMT -> Custom:SW_TS04-66-50-BK-260-SMT
- U3: footprint EasyEDA:TSSOP-8_L4.4-W3.0-P0.65-LS6.4-BL -> Custom:TSSOP-8_L4.4-W3.0-P0.65-LS6.4-BL; symbol EasyEDA:SP3485EET -> Custom:SP3485EET
- U5: footprint EasyEDA:SC-70-5_L2.1-W1.3-P0.65-LS2.1-BR -> Custom:SC-70-5_L2.1-W1.3-P0.65-LS2.1-BR; symbol EasyEDA:SN74LV1T34DCKR -> Custom:SN74LV1T34DCKR
Connections:
- net +5V: now also U8.6 (VOUT)
- net GND: now also C16.2, U8.2 (GND), U8.3 (~{CE})
- net VBUS: now also C16.1, U8.1 (VIN)
- removed net Earth: J1.10 (Earth_Gnd)
- no-connect marks 14 -> 15
Other:
- note added: "USB-C connector is provided for loading firmware or troubleshooting. VBUS feeds +5V through U8, an LM66100 ideal diode, so the board can run from USB alone (bench bring-up). When the IRM-05-5 is powered, U8 blocks reverse current into the host."
- note removed: "USB-C connector is provided for loading firmware or troubleshooting. This connector does *not* connect VBUS to the circuit. You cannot power the board from this connector nor receive power. Only the USB data D- and D+ pins are connected."
- moved on the sheet: C13, J4, J5, R11, R12, U7
