File: hardware/board/ecoport-bridge-v1/ecoport-bridge-v1.kicad_sch (KiCad schematic)
At the start: 64 parts, among them J1 420B2V12FL0, J2 Conn_01x02, J3 SM04B-SRSS-TB, J4 USB4085-GF-A, J5 Conn_01x02, J6 Connector Wire, J7 B3B-PH-K-S, SW1 RESET, SW2 BOOT, U1 IRM-05-5, U2 TLV75733PDBVR, U3 SP3485EET, U4 USBLC6-2SC6, U5 SN74LV1T34DCKR, U6 ESP32-C6-WROOM-1-N8, U7 USBLC6-2SC6, U8 LM66100DCKR

Commit message: Pull J1 pin 9, fill in MPNs, 1A fuse, rev-a release assets
- Remove J1 pin 9 (NC) from symbol, footprint and board: its floating pad
  sat 4.4 mm from F1 and 1.6 mm from pin 8, short of 5.5 mm creepage.
  Pull list is now pins 4, 6, 9, 10, 11.
- F1 to SF-2410SP100W-2 (1 A time-lag) for inrush margin; footprint fields
  and assembly notes updated to match.
- J3 is the top-entry BM04B-SRSS-TB to match its footprint.
- Add missing MPN/Manufacturer for U6, J7, J3, D2/D3 (value typo SKC6812 ->
  SK6812) and TP14, and include TP14 in the BOM.
- hardware/rev-a: populated bom.csv, DigiKey upload file for 6 boards,
  interactive BOM, board STEP for the enclosure (3d/), images/ for visual
  assets, and a README describing the folder.
- .gitignore: STEP and bom/ exports next to the KiCad project.

Co-Authored-By: Claude Opus 5.5 <noreply@anthropic.com>
Parts:
- D2, D3: value SKC6812 -> SK6812; MPN (none) -> SK6812; Manufacturer (none) -> OPSCO Optoelectronics
- F1: value SF-2410SP050W-2 -> SF-2410SP100W-2; Arrow Part Number SF-2410SP050W-2 -> SF-2410SP100W-2; Arrow Price/Stock https://www.arrow.com/en/products/sf-2410sp050w-2/bourns?re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 -> https://www.arrow.com/en/products/sf-2410sp100w-2/bourns?re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; MPN (none) -> SF-2410SP100W-2; Manufacturer (none) -> Bourns; Manufacturer_Part_Number SF-2410SP050W-2 -> SF-2410SP100W-2; Mouser Part Number 652-SF-2410SP050W-2 -> 652-SF-2410SP100W-2; Mouser Price/Stock https://www.mouser.co.uk/ProductDetail/Bourns/SF-2410SP050W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 -> https://www.mouser.co.uk/ProductDetail/Bourns/SF-2410SP100W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
- J3: value SM04B-SRSS-TB -> BM04B-SRSS-TB; MPN (none) -> BM04B-SRSS-TB(LF)(SN); Manufacturer (none) -> JST Sales America Inc.
- J7: MPN (none) -> B3B-PH-K-S(LF)(SN); Manufacturer (none) -> JST Sales America Inc.
- TP14: MPN (none) -> 5000; Manufacturer (none) -> Keystone; now in the parts list
- U6: MPN (none) -> ESP32-C6-WROOM-1-N8; Manufacturer (none) -> Espressif Systems
Changed lines of the file:
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@@
 		(pin "7"
 		)
-		(pin "9"
-		)
 		(pin "8"
 		)
@@
 			)
 		)
-		(property "Value" "SM04B-SRSS-TB"
+		(property "Value" "BM04B-SRSS-TB"
 			(at 43.18 142.24 0)
 			(show_name no)
@@
 			)
 		)
+		(property "Manufacturer" "JST Sales America Inc."
+			(at 0 0 0)
+			(hide yes)
+			(show_name no)
+			(do_not_autoplace no)
+			(effects
+				(font
+					(size 1.27 1.27)
+				)
+			)
+		)
+		(property "MPN" "BM04B-SRSS-TB(LF)(SN)"
+			(at 0 0 0)
+			(hide yes)
+			(show_name no)
+			(do_not_autoplace no)
+			(effects
+				(font
+					(size 1.27 1.27)
+				)
+			)
+		)
 		(pin "1"
 		)
@@
 		(body_style 1)
 		(exclude_from_sim no)
-		(in_bom no)
+		(in_bom yes)
 		(on_board yes)
 		(in_pos_files yes)
@@
 			)
 		)
+		(property "Manufacturer" "Keystone"
+			(at 0 0 0)
+			(hide yes)
+			(show_name no)
+			(do_not_autoplace no)
+			(effects
+				(font
+					(size 1.27 1.27)
+				)
+			)
+		)
+		(property "MPN" "5000"
+			(at 0 0 0)
+			(hide yes)
+			(show_name no)
+			(do_not_autoplace no)
+			(effects
+				(font
+					(size 1.27 1.27)
+				)
+			)
+		)
 		(pin "1"
 		)
@@
 			)
 		)
-		(property "Value" "SKC6812"
+		(property "Value" "SK6812"
 			(at 154.178 148.5198 0)
 			(show_name no)
@@
 			)
 		)
+		(property "Manufacturer" "OPSCO Optoelectronics"
+			(at 0 0 0)
+			(hide yes)
+			(show_name no)
+			(do_not_autoplace no)
+			(effects
+				(font
+					(size 1.27 1.27)
+				)
+			)
+		)
+		(property "MPN" "SK6812"
+			(at 0 0 0)
+			(hide yes)
+			(show_name no)
+			(do_not_autoplace no)
+			(effects
+				(font
+					(size 1.27 1.27)
+				)
+			)
+		)
 		(pin "3"
 		)
@@
 			)
 		)
-		(property "Value" "SKC6812"
+		(property "Value" "SK6812"
 			(at 156.21 159.004 0)
 			(show_name no)
@@
 			)
 		)
+		(property "Manufacturer" "OPSCO Optoelectronics"
+			(at 0 0 0)
+			(hide yes)
+			(show_name no)
+			(do_not_autoplace no)
+			(effects
+				(font
+					(size 1.27 1.27)
+				)
+			)
+		)
+		(property "MPN" "SK6812"
+			(at 0 0 0)
+			(hide yes)
+			(show_name no)
+			(do_not_autoplace no)
+			(effects
+				(font
+					(size 1.27 1.27)
+				)
+			)
+		)
 		(pin "3"
 		)
@@
 			)
 		)
+		(property "Manufacturer" "Espressif Systems"
+			(at 0 0 0)
+			(hide yes)
+			(show_name no)
+			(do_not_autoplace no)
+			(effects
+				(font
+					(size 1.27 1.27)
+				)
+			)
+		)
+		(property "MPN" "ESP32-C6-WROOM-1-N8"
+			(at 0 0 0)
+			(hide yes)
+			(show_name no)
+			(do_not_autoplace no)
+			(effects
+				(font
+					(size 1.27 1.27)
+				)
+			)
+		)
 		(pin "17"
 		)
@@
 			)
 		)
+		(property "Manufacturer" "JST Sales America Inc."
+			(at 0 0 0)
+			(hide yes)
+			(show_name no)
+			(do_not_autoplace no)
+			(effects
+				(font
+					(size 1.27 1.27)
+				)
+			)
+		)
+		(property "MPN" "B3B-PH-K-S(LF)(SN)"
+			(at 0 0 0)
+			(hide yes)
+			(show_name no)
+			(do_not_autoplace no)
+			(effects
+				(font
+					(size 1.27 1.27)
+				)
+			)
+		)
 		(pin "1"
 		)
@@
 			)
 		)
-		(property "Value" "SF-2410SP050W-2"
+		(property "Value" "SF-2410SP100W-2"
 			(at 76.2 66.04 0)
 			(show_name no)
@@
 			)
 		)
-		(property "Description" "Surface Mount Fuses 0.5A Time Lag 2410 SinglFuse"
+		(property "Description" "Surface Mount Fuses 1A Time Lag 2410 SinglFuse"
 			(at 76.2 48.26 0)
 			(hide yes)
@@
 			)
 		)
-		(property "Manufacturer_Part_Number" "SF-2410SP050W-2"
+		(property "Manufacturer_Part_Number" "SF-2410SP100W-2"
 			(at 76.2 55.88 0)
 			(hide yes)
@@
 			)
 		)
-		(property "Mouser Part Number" "652-SF-2410SP050W-2"
+		(property "Mouser Part Number" "652-SF-2410SP100W-2"
 			(at 76.2 58.42 0)
 			(hide yes)
@@
 			)
 		)
-		(property "Mouser Price/Stock" "https://www.mouser.co.uk/ProductDetail/Bourns/SF-2410SP050W-2?qs=55YtniHzbhAbLtmcAyIlLQ%3D%3D"
+		(property "Mouser Price/Stock" "https://www.mouser.co.uk/ProductDetail/Bourns/SF-2410SP100W-2"
 			(at 76.2 60.96 0)
 			(hide yes)
@@
 			)
 		)
-		(property "Arrow Part Number" "SF-2410SP050W-2"
+		(property "Arrow Part Number" "SF-2410SP100W-2"
 			(at 76.2 63.5 0)
 			(hide yes)
@@
 			)
 		)
-		(property "Arrow Price/Stock" "https://www.arrow.com/en/products/sf-2410sp050w-2/bourns?region=nac"
+		(property "Arrow Price/Stock" "https://www.arrow.com/en/products/sf-2410sp100w-2/bourns?region=nac"
 			(at 76.2 66.04 0)
 			(hide yes)
 			(show_name no)
+			(do_not_autoplace no)
+			(effects
+				(font
+					(size 1.27 1.27)
+				)
+			)
+		)
+		(property "Manufacturer" "Bourns"
+			(at 0 0 0)
+			(hide yes)
+			(show_name no)
+			(do_not_autoplace no)
+			(effects
+				(font
+					(size 1.27 1.27)
+				)
+			)
+		)
+		(property "MPN" "SF-2410SP100W-2"
+			(at 0 0 0)
+			(hide yes)
+			(show_name no)
