File: hardware/board/ecoport-bridge-v1/ecoport-bridge-v1.kicad_pcb (KiCad board)
At the start: 2 copper layers, 51.5 x 92 mm, 73 parts, among them J1 420B2V12FL0, J2 Conn_01x02, J3 BM04B-SRSS-TB, J4 USB4085-GF-A, J5 Conn_01x02, J6 Connector Wire, J7 B3B-PH-K-S, SW1 RESET, SW2 BOOT, U1 IRM-05-5, U2 TLV75733PDBVR, U3 SP3485EET, U4 USBLC6-2SC6, U5 SN74LV1T34DCKR, U6 ESP32-C6-WROOM-1-N8, U7 USBLC6-2SC6, U8 LM66100DCKR

Commit message: Graphics updates
Parts:
- added G***: EcoPort_Bridge_Marking, Custom:EcoPort_Bridge_Marking, B.Cu at (91.9, 113.7)
